Commit message: TF tree + topic namespacing for multi-robot verfication

File: urdf/gazebo_control.xacro (robot description, xacro)
@@ -45,5 +45,5 @@
             <joint_name>gimbal_pan_joint</joint_name>
             <joint_name>gimbal_tilt_joint</joint_name>
-            <topic>joint_states</topic>
+            <topic>${topic_prefix}/joint_states</topic>
             <update_rate>50</update_rate>
         </plugin>

File: urdf/gimbal.xacro (robot description, xacro)
@@ -145,3 +145,17 @@
     <origin xyz="0 0.03 ${tilt_z/2+0.025}" rpy="0 0 0" />
   </joint>
+  <!-- RGB Camera Optical Frame -->
+  <link name="gimbal_camera_optical_frame" />
+  <joint name="gimbal_camera_optical_joint" type="fixed">
+    <parent link="gimbal_camera_link" />
+    <child link="gimbal_camera_optical_frame" />
+    <origin xyz="0 0 0" rpy="${-pi/2} 0 ${-pi/2}" />
+  </joint>
+  <!-- IR Camera Optical Frame -->
+  <link name="gimbal_ir_camera_optical_frame" />
+  <joint name="gimbal_ir_camera_optical_joint" type="fixed">
+    <parent link="gimbal_ir_camera_link" />
+    <child link="gimbal_ir_camera_optical_frame" />
+    <origin xyz="0 0 0" rpy="${-pi/2} 0 ${-pi/2}" />
+  </joint>
 </robot>

File: urdf/sensors.xacro (robot description, xacro)
@@ -1,4 +1,9 @@
 <?xml version="1.0"?>
 <robot xmlns:xacro="http://www.ros.org/wiki/xacro" name="tin3_bot">
+    <!-- Add namespace properties at top of sensors.xacro -->
+    <xacro:arg name="robot_ns" default="" />
+    <xacro:property name="ns" value="$(arg robot_ns)" />
+    <xacro:property name="topic_prefix" value="${'/' + ns if ns != '' else ''}" />
+    <xacro:property name="frame_prefix" value="${ns + '/' if ns != '' else ''}" />
     <!-- ==================== -->
     <!-- GPS SENSOR           -->
@@ -22,6 +27,8 @@
             <always_on>true</always_on>
             <update_rate>5</update_rate>
-            <topic>/gps/fix</topic>
-            <gz_frame_id>gps_link</gz_frame_id>
+            <!-- <topic>/gps/fix</topic> -->
+            <!-- <gz_frame_id>gps_link</gz_frame_id> -->
+            <topic>${topic_prefix}/gps/fix</topic>
+            <gz_frame_id>${frame_prefix}gps_link</gz_frame_id>
             <navsat>
                 <position_sensing>
@@ -62,6 +69,8 @@
             <always_on>true</always_on>
             <update_rate>100</update_rate>
-            <topic>/imu/data</topic>
-            <gz_frame_id>imu_link</gz_frame_id>
+            <!-- <topic>/imu/data</topic> -->
+            <!-- <gz_frame_id>imu_link</gz_frame_id> -->
+             <topic>${topic_prefix}/imu/data</topic>
+            <gz_frame_id>${frame_prefix}imu_link</gz_frame_id>
             <imu>
                 <angular_velocity>
@@ -140,6 +149,8 @@
             <always_on>true</always_on>
             <update_rate>10</update_rate>
-            <topic>/scan</topic>
-            <gz_frame_id>lidar_link</gz_frame_id>
+            <!-- <topic>/scan</topic> -->
+            <!-- <gz_frame_id>lidar_link</gz_frame_id> -->
+            <topic>${topic_prefix}/scan</topic>
+            <gz_frame_id>${frame_prefix}lidar_link</gz_frame_id>
             <lidar>
                 <scan>
@@ -178,6 +189,8 @@
             <always_on>true</always_on>
             <update_rate>30</update_rate>
-            <topic>/camera/image_raw</topic>
-            <gz_frame_id>gimbal_camera_link</gz_frame_id>
+            <!-- <topic>/camera/image_raw</topic> -->
+            <!-- <gz_frame_id>gimbal_camera_link</gz_frame_id> -->
+             <topic>${topic_prefix}/camera/image_raw</topic>
+            <gz_frame_id>${frame_prefix}gimbal_camera_link</gz_frame_id>
             <camera>
                 <horizontal_fov>1.047</horizontal_fov>
@@ -206,6 +219,8 @@
             <always_on>true</always_on>
             <update_rate>30</update_rate>
-            <topic>/ir/image_raw</topic>
-            <gz_frame_id>gimbal_ir_camera_link</gz_frame_id>
+            <!-- <topic>/ir/image_raw</topic> -->
+            <!-- <gz_frame_id>gimbal_ir_camera_link</gz_frame_id> -->
+             <topic>${topic_prefix}/ir/image_raw</topic>
+            <gz_frame_id>${frame_prefix}gimbal_ir_camera_link</gz_frame_id>
             <camera>
                 <horizontal_fov>1.047</horizontal_fov>
