Commit message: Week 1 complete: URDF, physics, diff drive, launch files
- Centered chassis and track meshes
- URDF with proper TF tree (base_footprint → base_link → wheels/tracks)
- Gazebo friction parameters for tracks
- Differential drive plugin (6 wheel joints)
- Joint state publisher plugin
- Launch files: spawn_robot, tin3_gz, multi_robot
- Robot moves via cmd_vel, odom publishing works
- Multi-robot spawning with namespace support

File: urdf/robot.urdf.xacro (robot description, xacro)
@@ -3,41 +3,30 @@
   <!-- Include materials -->
   <xacro:include filename="$(find tin3_bot)/urdf/materials.xacro"/>
+   <xacro:include filename="$(find tin3_bot)/urdf/gazebo.xacro"/>
+   <xacro:include filename="$(find tin3_bot)/urdf/gazebo_control.xacro"/>
   <!-- ==================== -->
   <!-- PROPERTIES (meters)  -->
   <!-- ==================== -->
-  <!-- Mesh scale: 1 1 1 (meshes already in correct units) -->
+  <!-- Mesh scale: 0.001 to convert mm to meters -->
   <xacro:property name="mesh_scale" value="1 1 1"/>
-  <!-- Chassis dimensions (from BoundBox, in meters) -->
+  <!-- Chassis dimensions (meters) -->
   <xacro:property name="chassis_length" value="0.837"/>
   <xacro:property name="chassis_width" value="1.314"/>
   <xacro:property name="chassis_height" value="0.606"/>
   <xacro:property name="chassis_mass" value="20.0"/>
-  <!-- Track dimensions (from BoundBox, in meters) -->
-  <xacro:property name="track_thickness" value="0.150"/>
-  <xacro:property name="track_length" value="1.214"/>
-  <xacro:property name="track_height" value="0.334"/>
-  <!--
-    TRACK OFFSETS - Adjust these independently for left and right tracks
-    Positive X = left side of robot
-    Negative X = right side of robot
-  -->
-  <xacro:property name="left_track_x_offset" value="0.5"/>
-  <xacro:property name="right_track_x_offset" value="-0.19"/>
-  <!-- Track Y offset (front/back adjustment if needed) -->
-  <xacro:property name="left_track_y_offset" value="-0.1"/>
-  <xacro:property name="right_track_y_offset" value="-0.1"/>
-  <!-- Track Z offset (vertical position) -->
-  <xacro:property name="left_track_z_offset" value="0.06"/>
-  <xacro:property name="right_track_z_offset" value="0.06"/>
+  <!-- Track offsets from base_link center (meters) -->
+  <xacro:property name="track_y_offset" value="0.35"/>
+  <xacro:property name="track_z_offset" value="-0.22"/>
   <!-- Hidden wheel parameters -->
   <xacro:property name="wheel_radius" value="0.12"/>
   <xacro:property name="wheel_width" value="0.10"/>
   <xacro:property name="wheel_mass" value="1.0"/>
-  <!-- Wheel positions along track (Y direction = front/back) -->
-  <xacro:property name="wheel_front_y" value="0.40"/>
-  <xacro:property name="wheel_mid_y" value="0.0"/>
-  <xacro:property name="wheel_rear_y" value="-0.40"/>
+  <!-- Wheel positions along track (X direction = front/back) -->
+  <xacro:property name="wheel_front_x" value="0.40"/>
+  <xacro:property name="wheel_mid_x" value="0.0"/>
+  <xacro:property name="wheel_rear_x" value="-0.40"/>
   <!-- Wheel Z position (below base_link origin) -->
-  <xacro:property name="wheel_z" value="-0.15"/>
+  <!-- <xacro:property name="wheel_z" value="-0.15"/> -->
+<xacro:property name="wheel_z" value="-0.27"/>
   <!-- ==================== -->
   <!-- MACROS               -->
@@ -55,35 +44,36 @@
              izz="${m*r*r/2}"/>
   </xacro:macro>
-<!-- Macro for hidden wheel -->
-<xacro:macro name="hidden_wheel" params="name x_pos y_pos z_pos">
-  <link name="${name}">
-    <collision>
-      <origin xyz="0 0 0" rpy="${pi/2} 0 0"/>
-      <geometry>
-        <cylinder radius="${wheel_radius}" length="${wheel_width}"/>
-      </geometry>
-    </collision>
-    <inertial>
-      <origin xyz="0 0 0" rpy="${pi/2} 0 0"/>
-      <mass value="${wheel_mass}"/>
-      <xacro:cylinder_inertia m="${wheel_mass}" r="${wheel_radius}" l="${wheel_width}"/>
-    </inertial>
-  </link>
-  <joint name="${name}_joint" type="continuous">
-    <parent link="base_link"/>
-    <child link="${name}"/>
-    <origin xyz="${x_pos} ${y_pos} ${z_pos}" rpy="0 0 ${-pi/2}"/>
-    <axis xyz="0 1 0"/>
+  <!-- Macro for hidden wheel -->
+  <xacro:macro name="hidden_wheel" params="name x_pos y_pos z_pos">
+    <link name="${name}">
+      <collision>
+        <origin xyz="0 0 0" rpy="${pi/2} 0 0"/>
+        <geometry>
+          <cylinder radius="${wheel_radius}" length="${wheel_width}"/>
+        </geometry>
+      </collision>
+      <inertial>
+        <origin xyz="0 0 0" rpy="0 0 0"/>
+        <mass value="${wheel_mass}"/>
+        <xacro:cylinder_inertia m="${wheel_mass}" r="${wheel_radius}" l="${wheel_width}"/>
+      </inertial>
+    </link>
+    <joint name="${name}_joint" type="continuous">
+      <parent link="base_link"/>
+      <child link="${name}"/>
+      <origin xyz="${x_pos} ${y_pos} ${z_pos}" rpy="0 0 0"/>
+      <axis xyz="0 1 0"/>
+    </joint>
+  </xacro:macro>
+  <!-- ==================== -->
+  <!-- BASE FOOTPRINT       -->
+  <!-- ==================== -->
+  <link name="base_footprint"/>
+  <joint name="base_footprint_joint" type="fixed">
+    <parent link="base_footprint"/>
+    <child link="base_link"/>
+    <!-- <origin xyz="0 0 0.27" rpy="0 0 0"/> -->
+       <origin xyz="0 0 0.387" rpy="0 0 0"/>
   </joint>
-</xacro:macro>
-<!-- ==================== -->
-<!-- BASE FOOTPRINT       -->
-<!-- ==================== -->
-<link name="base_footprint"/>
-<joint name="base_footprint_joint" type="fixed">
-  <parent link="base_footprint"/>
-  <child link="base_link"/>
-  <origin xyz="0 0 0.27" rpy="0 0 0"/>
-</joint>
   <!-- ==================== -->
   <!-- BASE LINK (CHASSIS)  -->
@@ -91,5 +81,5 @@
   <link name="base_link">
     <visual>
-      <origin xyz="0 0 0" rpy="0 0 0"/>
+      <origin xyz="0 0 0" rpy="0 0 ${pi/2}"/>
       <geometry>
         <mesh filename="package://tin3_bot/meshes/chassis.dae" scale="${mesh_scale}"/>
@@ -97,13 +87,13 @@
       <material name="dark_gray"/>
     </visual>
-    <collision>
+    <!-- <collision>
+      <origin xyz="0 0 0" rpy="0 0 0"/>
       <geometry>
         <box size="${chassis_length} ${chassis_width} ${chassis_height}"/>
       </geometry>
-      <origin xyz="0 0 ${chassis_height/2}" rpy="0 0 0"/>
-    </collision>
+    </collision> -->
     <inertial>
+      <origin xyz="0 0 0" rpy="0 0 0"/>
       <mass value="${chassis_mass}"/>
-      <origin xyz="0 0 ${chassis_height/2}" rpy="0 0 0"/>
       <xacro:box_inertia m="${chassis_mass}" x="${chassis_length}" y="${chassis_width}" z="${chassis_height}"/>
     </inertial>
@@ -115,5 +105,5 @@
   <link name="left_track_visual">
     <visual>
-        <origin xyz="0 0 0" rpy="0 0 ${pi/2}"/>
+      <origin xyz="0 0 0" rpy="0 0 ${-pi/2}"/>
       <geometry>
         <mesh filename="package://tin3_bot/meshes/left_track.dae" scale="${mesh_scale}"/>
@@ -129,10 +119,10 @@
     <parent link="base_link"/>
     <child link="left_track_visual"/>
-    <origin xyz="${left_track_x_offset} ${left_track_y_offset} ${left_track_z_offset}" rpy="0 0 ${-pi/2}"/>
+    <origin xyz="0 ${track_y_offset} ${track_z_offset}" rpy="0 0 0"/>
   </joint>
   <!-- Right Track Visual -->
   <link name="right_track_visual">
     <visual>
-        <origin xyz="0 0 0" rpy="0 0 ${pi/2}"/>
+      <origin xyz="0 0 0" rpy="0 0 ${-pi/2}"/>
       <geometry>
         <mesh filename="package://tin3_bot/meshes/right_track.dae" scale="${mesh_scale}"/>
@@ -148,5 +138,5 @@
     <parent link="base_link"/>
     <child link="right_track_visual"/>
-    <origin xyz="${right_track_x_offset} ${right_track_y_offset} ${right_track_z_offset}" rpy="0 0 ${-pi/2}"/>
+    <origin xyz="0 ${-track_y_offset} ${track_z_offset}" rpy="0 0 0"/>
   </joint>
   <!-- ==================== -->
@@ -155,27 +145,27 @@
   <!-- Left side wheels (3 wheels) -->
   <xacro:hidden_wheel name="left_front_wheel"
-                       x_pos="${left_track_x_offset}"
-                       y_pos="${wheel_front_y}"
+                       x_pos="${wheel_front_x}"
+                       y_pos="${track_y_offset}"
                        z_pos="${wheel_z}"/>
   <xacro:hidden_wheel name="left_mid_wheel"
-                       x_pos="${left_track_x_offset}"
-                       y_pos="${wheel_mid_y}"
+                       x_pos="${wheel_mid_x}"
+                       y_pos="${track_y_offset}"
                        z_pos="${wheel_z}"/>
   <xacro:hidden_wheel name="left_rear_wheel"
-                       x_pos="${left_track_x_offset}"
-                       y_pos="${wheel_rear_y}"
+                       x_pos="${wheel_rear_x}"
+                       y_pos="${track_y_offset}"
                        z_pos="${wheel_z}"/>
   <!-- Right side wheels (3 wheels) -->
   <xacro:hidden_wheel name="right_front_wheel"
-                       x_pos="${right_track_x_offset}"
-                       y_pos="${wheel_front_y}"
+                       x_pos="${wheel_front_x}"
+                       y_pos="${-track_y_offset}"
                        z_pos="${wheel_z}"/>
   <xacro:hidden_wheel name="right_mid_wheel"
-                       x_pos="${right_track_x_offset}"
-                       y_pos="${wheel_mid_y}"
+                       x_pos="${wheel_mid_x}"
+                       y_pos="${-track_y_offset}"
                        z_pos="${wheel_z}"/>
   <xacro:hidden_wheel name="right_rear_wheel"
-                       x_pos="${right_track_x_offset}"
-                       y_pos="${wheel_rear_y}"
+                       x_pos="${wheel_rear_x}"
+                       y_pos="${-track_y_offset}"
                        z_pos="${wheel_z}"/>
 </robot>

Commit message: add EKF,Nav2 integration and refactor launch files

File: urdf/robot.urdf.xacro (robot description, xacro)
@@ -89,7 +89,7 @@
     </visual>
     <!-- <collision>
-      <origin xyz="0 0 0" rpy="0 0 0"/>
+      <origin xyz="0 0 0" rpy="0 0 0" />
       <geometry>
-        <box size="${chassis_length} ${chassis_width} ${chassis_height}"/>
+        <box size="${chassis_length} ${chassis_width} ${chassis_height}" />
       </geometry>
     </collision> -->
@@ -120,4 +120,10 @@
       </geometry>
       <material name="dark_gray" />
+      <!-- <collision>
+        <origin xyz="0 0 0" rpy="0 0 0" />
+        <geometry>
+          <box size="0.8 0.15 0.24" />
+        </geometry>
+      </collision> -->
     </visual>
     <inertial>
@@ -139,4 +145,10 @@
       </geometry>
       <material name="dark_gray" />
+      <!-- <collision>
+        <origin xyz="0 0 0" rpy="0 0 0" />
+        <geometry>
+          <box size="0.8 0.15 0.24" />
+        </geometry>
+      </collision> -->
     </visual>
     <inertial>

File: urdf/sensors.xacro (robot description, xacro)
@@ -71,5 +71,5 @@
             <!-- <topic>/imu/data</topic> -->
             <!-- <gz_frame_id>imu_link</gz_frame_id> -->
-             <topic>${topic_prefix}/imu/data</topic>
+            <topic>${topic_prefix}/imu/data</topic>
             <gz_frame_id>${frame_prefix}imu_link</gz_frame_id>
             <imu>
@@ -149,6 +149,4 @@
             <always_on>true</always_on>
             <update_rate>10</update_rate>
-            <!-- <topic>/scan</topic> -->
-            <!-- <gz_frame_id>lidar_link</gz_frame_id> -->
             <topic>${topic_prefix}/scan</topic>
             <gz_frame_id>${frame_prefix}lidar_link</gz_frame_id>
@@ -156,19 +154,21 @@
                 <scan>
                     <horizontal>
-                        <samples>180</samples>
+                        <!-- FOV: 120° / 0.625° = 192 samples -->
+                        <samples>192</samples>
                         <resolution>1</resolution>
-                        <min_angle>-1.5708</min_angle>
-                        <max_angle>1.5708</max_angle>
+                        <min_angle>-1.0472</min_angle>  <!-- -60° -->
+                        <max_angle>1.0472</max_angle>   <!-- +60° -->
                     </horizontal>
                     <vertical>
-                        <samples>1</samples>
+                        <!-- FOV: 90° with 144 lines (per spec) -->
+                        <samples>144</samples>
                         <resolution>1</resolution>
-                        <min_angle>0</min_angle>
-                        <max_angle>0</max_angle>
+                        <min_angle>-0.7854</min_angle>  <!-- -45° -->
+                        <max_angle>0.7854</max_angle>   <!-- +45° -->
                     </vertical>
                 </scan>
                 <range>
                     <min>0.1</min>
-                    <max>30.0</max>
+                    <max>30.0</max>      <!-- 30m @ 10% reflectivity -->
                     <resolution>0.01</resolution>
                 </range>
@@ -176,5 +176,5 @@
                     <type>gaussian</type>
                     <mean>0.0</mean>
-                    <stddev>0.01</stddev>
+                    <stddev>0.05</stddev>  <!-- ±5cm accuracy -->
                 </noise>
             </lidar>
@@ -191,5 +191,5 @@
             <!-- <topic>/camera/image_raw</topic> -->
             <!-- <gz_frame_id>gimbal_camera_link</gz_frame_id> -->
-             <topic>${topic_prefix}/camera/image_raw</topic>
+            <topic>${topic_prefix}/camera/image_raw</topic>
             <gz_frame_id>${frame_prefix}gimbal_camera_link</gz_frame_id>
             <camera>
@@ -221,5 +221,5 @@
             <!-- <topic>/ir/image_raw</topic> -->
             <!-- <gz_frame_id>gimbal_ir_camera_link</gz_frame_id> -->
-             <topic>${topic_prefix}/ir/image_raw</topic>
+            <topic>${topic_prefix}/ir/image_raw</topic>
             <gz_frame_id>${frame_prefix}gimbal_ir_camera_link</gz_frame_id>
             <camera>
