Commit message: fix: collision and inertia consistency

File: urdf/gimbal.xacro (robot description, xacro)
@@ -32,9 +32,4 @@
       </geometry>
     </visual>
-    <!-- <collision>
-      <geometry>
-        <box size="0.172 0.180 0.194" />
-      </geometry>
-    </collision> -->
     <collision>
       <geometry>
@@ -44,5 +39,5 @@
     <inertial>
       <mass value="0.8" />
-      <inertia ixx="0.002" ixy="0" ixz="0" iyy="0.002" iyz="0" izz="0.002" />
+       <inertia ixx="0.003" ixy="0" ixz="0" iyy="0.003" iyz="0" izz="0.003" />
     </inertial>
   </link>
@@ -63,17 +58,12 @@
       </geometry>
     </visual>
-    <!-- <collision>
-      <geometry>
-        <box size="0.125 0.218 0.211" />
-      </geometry>
-    </collision> -->
     <collision>
       <geometry>
-        <box size="0.10 0.18 0.15" />  <!-- Smaller -->
+        <box size="0.10 0.18 0.15" />
       </geometry>
     </collision>
     <inertial>
       <mass value="0.5" />
-      <inertia ixx="0.001" ixy="0" ixz="0" iyy="0.001" iyz="0" izz="0.001" />
+      <inertia ixx="0.0023" ixy="0" ixz="0" iyy="0.0014" iyz="0" izz="0.0018" />
     </inertial>
   </link>
@@ -136,5 +126,5 @@
     </collision>
     <inertial>
-      <mass value="0.2" />
+      <mass value="0.05" />
       <inertia ixx="0.0001" ixy="0" ixz="0" iyy="0.0001" iyz="0" izz="0.0001" />
     </inertial>

File: urdf/robot.urdf.xacro (robot description, xacro)
@@ -88,10 +88,10 @@
       <material name="dark_gray" />
     </visual>
-    <!-- <collision>
+    <collision>
       <origin xyz="0 0 0" rpy="0 0 0" />
       <geometry>
-        <box size="${chassis_length} ${chassis_width} ${chassis_height}" />
+         <box size="1.32 0.55 0.49" />
       </geometry>
-    </collision> -->
+    </collision>
     <inertial>
       <origin xyz="0 0 0" rpy="0 0 0" />
@@ -120,11 +120,12 @@
       </geometry>
       <material name="dark_gray" />
-      <!-- <collision>
-        <origin xyz="0 0 0" rpy="0 0 0" />
-        <geometry>
-          <box size="0.8 0.15 0.24" />
-        </geometry>
-      </collision> -->
     </visual>
+    <collision>
+      <origin xyz="0 0 0" rpy="0 0 0" />
+      <geometry>
+        <!-- <box size="0.8 0.15 0.24" /> -->
+          <box size="1.22 0.154 0.33" />
+      </geometry>
+    </collision>
     <inertial>
       <mass value="0.01" />
@@ -145,11 +146,12 @@
       </geometry>
       <material name="dark_gray" />
-      <!-- <collision>
-        <origin xyz="0 0 0" rpy="0 0 0" />
-        <geometry>
-          <box size="0.8 0.15 0.24" />
-        </geometry>
-      </collision> -->
     </visual>
+    <collision>
+      <origin xyz="0 0 0" rpy="0 0 0" />
+      <geometry>
+        <!-- <box size="0.8 0.15 0.24" /> -->
+        <box size="1.22 0.154 0.33" />
+      </geometry>
+    </collision>
     <inertial>
       <mass value="0.01" />
