Commit message: Week 2:Sensor integration complete

File: urdf/gazebo.xacro (robot description, xacro)
@@ -16,10 +16,10 @@
   </xacro:macro>
   <!-- Apply friction to all hidden wheels -->
-  <xacro:wheel_friction wheel_name="left_front_wheel"/>
-  <xacro:wheel_friction wheel_name="left_mid_wheel"/>
-  <xacro:wheel_friction wheel_name="left_rear_wheel"/>
-  <xacro:wheel_friction wheel_name="right_front_wheel"/>
-  <xacro:wheel_friction wheel_name="right_mid_wheel"/>
-  <xacro:wheel_friction wheel_name="right_rear_wheel"/>
+  <xacro:wheel_friction wheel_name="left_front_wheel" />
+  <xacro:wheel_friction wheel_name="left_mid_wheel" />
+  <xacro:wheel_friction wheel_name="left_rear_wheel" />
+  <xacro:wheel_friction wheel_name="right_front_wheel" />
+  <xacro:wheel_friction wheel_name="right_mid_wheel" />
+  <xacro:wheel_friction wheel_name="right_rear_wheel" />
   <!-- ==================== -->
   <!-- GAZEBO MATERIALS     -->
@@ -34,3 +34,9 @@
     <material>Gazebo/Black</material>
   </gazebo>
+  <gazebo reference="gimbal_pan_link">
+    <self_collide>false</self_collide>
+  </gazebo>
+  <gazebo reference="gimbal_tilt_link">
+    <self_collide>false</self_collide>
+  </gazebo>
 </robot>

File: urdf/gazebo_control.xacro (robot description, xacro)
@@ -1,4 +1,11 @@
 <?xml version="1.0"?>
 <robot xmlns:xacro="http://www.ros.org/wiki/xacro">
+    <!-- Namespace argument -->
+    <xacro:arg name="robot_ns" default="" />
+    <xacro:property name="ns" value="$(arg robot_ns)" />
+    <!-- Topic prefix: /ns or empty for topics -->
+    <xacro:property name="topic_prefix" value="${'/' + ns if ns != '' else ''}" />
+    <!-- Frame prefix: ns/ or empty for frame_ids (no leading slash) -->
+    <xacro:property name="frame_prefix" value="${ns + '/' if ns != '' else ''}" />
     <!-- ==================== -->
     <!-- DIFFERENTIAL DRIVE   -->
@@ -20,13 +27,14 @@
             <max_linear_acceleration>0.5</max_linear_acceleration>
             <max_angular_acceleration>1.0</max_angular_acceleration>
-            <!-- Topics -->
-            <topic>cmd_vel</topic>
-            <odom_topic>odom</odom_topic>
-            <tf_topic>tf</tf_topic>
-            <frame_id>odom</frame_id>
-            <child_frame_id>base_footprint</child_frame_id>
+            <!-- Topics with namespace -->
+            <topic>${topic_prefix}/cmd_vel</topic>
+            <odom_topic>${topic_prefix}/odom</odom_topic>
+            <tf_topic>${topic_prefix}/tf</tf_topic>
+            <frame_id>${frame_prefix}odom</frame_id>
+            <child_frame_id>${frame_prefix}base_footprint</child_frame_id>
             <odom_publish_frequency>50</odom_publish_frequency>
         </plugin>
-        <plugin filename="gz-sim-joint-state-publisher-system" name="gz::sim::systems::JointStatePublisher">
+        <plugin filename="gz-sim-joint-state-publisher-system"
+            name="gz::sim::systems::JointStatePublisher">
             <joint_name>left_front_wheel_joint</joint_name>
             <joint_name>left_mid_wheel_joint</joint_name>
@@ -35,5 +43,39 @@
             <joint_name>right_mid_wheel_joint</joint_name>
             <joint_name>right_rear_wheel_joint</joint_name>
+            <joint_name>gimbal_pan_joint</joint_name>
+            <joint_name>gimbal_tilt_joint</joint_name>
             <topic>joint_states</topic>
+            <update_rate>50</update_rate>
+        </plugin>
+    </gazebo>
+    <!-- ==================== -->
+    <!-- GIMBAL CONTROLLERS   -->
+    <!-- ==================== -->
+    <!-- Gimbal Pan Controller -->
+    <gazebo>
+        <plugin filename="gz-sim-joint-position-controller-system"
+            name="gz::sim::systems::JointPositionController">
+            <joint_name>gimbal_pan_joint</joint_name>
+            <topic>${topic_prefix}/gimbal/pan_cmd</topic>
+            <!-- <p_gain>10</p_gain>
+            <i_gain>0.1</i_gain>
+            <d_gain>0.5</d_gain> -->
+            <p_gain>5</p_gain>
+            <i_gain>0.0</i_gain>
+            <d_gain>1.0</d_gain>
+        </plugin>
+    </gazebo>
+    <!-- Gimbal Tilt Controller -->
+    <gazebo>
+        <plugin filename="gz-sim-joint-position-controller-system"
+            name="gz::sim::systems::JointPositionController">
+            <joint_name>gimbal_tilt_joint</joint_name>
+            <topic>${topic_prefix}/gimbal/tilt_cmd</topic>
+            <!-- <p_gain>10</p_gain>
+            <i_gain>0.1</i_gain>
+            <d_gain>0.5</d_gain> -->
+            <p_gain>5</p_gain>
+            <i_gain>0.0</i_gain>
+            <d_gain>1.0</d_gain>
         </plugin>
     </gazebo>

File: urdf/robot.urdf.xacro (robot description, xacro)
@@ -1,32 +1,33 @@
 <?xml version="1.0"?>
 <robot xmlns:xacro="http://www.ros.org/wiki/xacro" name="tin3_bot">
-  <!-- Include materials -->
-  <xacro:include filename="$(find tin3_bot)/urdf/materials.xacro"/>
-   <xacro:include filename="$(find tin3_bot)/urdf/gazebo.xacro"/>
-   <xacro:include filename="$(find tin3_bot)/urdf/gazebo_control.xacro"/>
+  <xacro:include filename="$(find tin3_bot)/urdf/materials.xacro" />
+  <xacro:include filename="$(find tin3_bot)/urdf/gazebo.xacro" />
+  <xacro:include filename="$(find tin3_bot)/urdf/gazebo_control.xacro" />
+  <xacro:include filename="$(find tin3_bot)/urdf/gimbal.xacro" />
+  <xacro:include filename="$(find tin3_bot)/urdf/sensors.xacro" />
   <!-- ==================== -->
   <!-- PROPERTIES (meters)  -->
   <!-- ==================== -->
   <!-- Mesh scale: 0.001 to convert mm to meters -->
-  <xacro:property name="mesh_scale" value="1 1 1"/>
+  <xacro:property name="mesh_scale" value="1 1 1" />
   <!-- Chassis dimensions (meters) -->
-  <xacro:property name="chassis_length" value="0.837"/>
-  <xacro:property name="chassis_width" value="1.314"/>
-  <xacro:property name="chassis_height" value="0.606"/>
-  <xacro:property name="chassis_mass" value="20.0"/>
+  <xacro:property name="chassis_length" value="0.837" />
+  <xacro:property name="chassis_width" value="1.314" />
+  <xacro:property name="chassis_height" value="0.606" />
+  <xacro:property name="chassis_mass" value="20.0" />
   <!-- Track offsets from base_link center (meters) -->
-  <xacro:property name="track_y_offset" value="0.35"/>
-  <xacro:property name="track_z_offset" value="-0.22"/>
+  <xacro:property name="track_y_offset" value="0.35" />
+  <xacro:property name="track_z_offset" value="-0.22" />
   <!-- Hidden wheel parameters -->
-  <xacro:property name="wheel_radius" value="0.12"/>
-  <xacro:property name="wheel_width" value="0.10"/>
-  <xacro:property name="wheel_mass" value="1.0"/>
+  <xacro:property name="wheel_radius" value="0.12" />
+  <xacro:property name="wheel_width" value="0.10" />
+  <xacro:property name="wheel_mass" value="1.0" />
   <!-- Wheel positions along track (X direction = front/back) -->
-  <xacro:property name="wheel_front_x" value="0.40"/>
-  <xacro:property name="wheel_mid_x" value="0.0"/>
-  <xacro:property name="wheel_rear_x" value="-0.40"/>
+  <xacro:property name="wheel_front_x" value="0.40" />
+  <xacro:property name="wheel_mid_x" value="0.0" />
+  <xacro:property name="wheel_rear_x" value="-0.40" />
   <!-- Wheel Z position (below base_link origin) -->
   <!-- <xacro:property name="wheel_z" value="-0.15"/> -->
-<xacro:property name="wheel_z" value="-0.27"/>
+  <xacro:property name="wheel_z" value="-0.27" />
   <!-- ==================== -->
   <!-- MACROS               -->
@@ -35,12 +36,12 @@
   <xacro:macro name="box_inertia" params="m x y z">
     <inertia ixx="${m*(y*y+z*z)/12}" ixy="0" ixz="0"
-             iyy="${m*(x*x+z*z)/12}" iyz="0"
-             izz="${m*(x*x+y*y)/12}"/>
+      iyy="${m*(x*x+z*z)/12}" iyz="0"
+      izz="${m*(x*x+y*y)/12}" />
   </xacro:macro>
   <!-- Macro for inertia of a cylinder -->
   <xacro:macro name="cylinder_inertia" params="m r l">
     <inertia ixx="${m*(3*r*r+l*l)/12}" ixy="0" ixz="0"
-             iyy="${m*(3*r*r+l*l)/12}" iyz="0"
-             izz="${m*r*r/2}"/>
+      iyy="${m*(3*r*r+l*l)/12}" iyz="0"
+      izz="${m*r*r/2}" />
   </xacro:macro>
   <!-- Macro for hidden wheel -->
@@ -48,20 +49,20 @@
     <link name="${name}">
       <collision>
-        <origin xyz="0 0 0" rpy="${pi/2} 0 0"/>
+        <origin xyz="0 0 0" rpy="${pi/2} 0 0" />
         <geometry>
-          <cylinder radius="${wheel_radius}" length="${wheel_width}"/>
+          <cylinder radius="${wheel_radius}" length="${wheel_width}" />
         </geometry>
       </collision>
       <inertial>
-        <origin xyz="0 0 0" rpy="0 0 0"/>
-        <mass value="${wheel_mass}"/>
-        <xacro:cylinder_inertia m="${wheel_mass}" r="${wheel_radius}" l="${wheel_width}"/>
+        <origin xyz="0 0 0" rpy="0 0 0" />
+        <mass value="${wheel_mass}" />
+        <xacro:cylinder_inertia m="${wheel_mass}" r="${wheel_radius}" l="${wheel_width}" />
       </inertial>
     </link>
     <joint name="${name}_joint" type="continuous">
-      <parent link="base_link"/>
-      <child link="${name}"/>
-      <origin xyz="${x_pos} ${y_pos} ${z_pos}" rpy="0 0 0"/>
-      <axis xyz="0 1 0"/>
+      <parent link="base_link" />
+      <child link="${name}" />
+      <origin xyz="${x_pos} ${y_pos} ${z_pos}" rpy="0 0 0" />
+      <axis xyz="0 1 0" />
     </joint>
   </xacro:macro>
@@ -69,10 +70,10 @@
   <!-- BASE FOOTPRINT       -->
   <!-- ==================== -->
-  <link name="base_footprint"/>
+  <link name="base_footprint" />
   <joint name="base_footprint_joint" type="fixed">
-    <parent link="base_footprint"/>
-    <child link="base_link"/>
+    <parent link="base_footprint" />
+    <child link="base_link" />
     <!-- <origin xyz="0 0 0.27" rpy="0 0 0"/> -->
-       <origin xyz="0 0 0.387" rpy="0 0 0"/>
+    <origin xyz="0 0 0.387" rpy="0 0 0" />
   </joint>
   <!-- ==================== -->
@@ -81,9 +82,9 @@
   <link name="base_link">
     <visual>
-      <origin xyz="0 0 0" rpy="0 0 ${pi/2}"/>
+      <origin xyz="0 0 0" rpy="0 0 ${pi/2}" />
       <geometry>
-        <mesh filename="package://tin3_bot/meshes/chassis.dae" scale="${mesh_scale}"/>
+        <mesh filename="package://tin3_bot/meshes/chassis.dae" scale="${mesh_scale}" />
       </geometry>
-      <material name="dark_gray"/>
+      <material name="dark_gray" />
     </visual>
     <!-- <collision>
@@ -94,9 +95,18 @@
     </collision> -->
     <inertial>
-      <origin xyz="0 0 0" rpy="0 0 0"/>
-      <mass value="${chassis_mass}"/>
-      <xacro:box_inertia m="${chassis_mass}" x="${chassis_length}" y="${chassis_width}" z="${chassis_height}"/>
+      <origin xyz="0 0 0" rpy="0 0 0" />
+      <mass value="${chassis_mass}" />
+      <xacro:box_inertia m="${chassis_mass}" x="${chassis_length}" y="${chassis_width}"
+        z="${chassis_height}" />
     </inertial>
   </link>
+  <!-- ==================== -->
+  <!-- Gimbal Joint        -->
+  <!-- ==================== -->
+  <joint name="gimbal_base_joint" type="fixed">
+    <parent link="base_link" />
+    <child link="gimbal_base_link" />
+    <origin xyz="0.1  0  0.303" rpy="0 0 0" />
+  </joint>
   <!-- ==================== -->
   <!-- TRACK VISUALS        -->
@@ -105,38 +115,38 @@
   <link name="left_track_visual">
     <visual>
-      <origin xyz="0 0 0" rpy="0 0 ${-pi/2}"/>
+      <origin xyz="0 0 0" rpy="0 0 ${-pi/2}" />
       <geometry>
-        <mesh filename="package://tin3_bot/meshes/left_track.dae" scale="${mesh_scale}"/>
+        <mesh filename="package://tin3_bot/meshes/left_track.dae" scale="${mesh_scale}" />
       </geometry>
-      <material name="dark_gray"/>
+      <material name="dark_gray" />
     </visual>
     <inertial>
-      <mass value="0.01"/>
-      <inertia ixx="0.0001" ixy="0" ixz="0" iyy="0.0001" iyz="0" izz="0.0001"/>
+      <mass value="0.01" />
+      <inertia ixx="0.0001" ixy="0" ixz="0" iyy="0.0001" iyz="0" izz="0.0001" />
     </inertial>
   </link>
   <joint name="left_track_visual_joint" type="fixed">
-    <parent link="base_link"/>
-    <child link="left_track_visual"/>
-    <origin xyz="0 ${track_y_offset} ${track_z_offset}" rpy="0 0 0"/>
+    <parent link="base_link" />
+    <child link="left_track_visual" />
+    <origin xyz="0 ${track_y_offset} ${track_z_offset}" rpy="0 0 0" />
   </joint>
   <!-- Right Track Visual -->
   <link name="right_track_visual">
     <visual>
-      <origin xyz="0 0 0" rpy="0 0 ${-pi/2}"/>
+      <origin xyz="0 0 0" rpy="0 0 ${-pi/2}" />
       <geometry>
-        <mesh filename="package://tin3_bot/meshes/right_track.dae" scale="${mesh_scale}"/>
+        <mesh filename="package://tin3_bot/meshes/right_track.dae" scale="${mesh_scale}" />
       </geometry>
-      <material name="dark_gray"/>
+      <material name="dark_gray" />
     </visual>
     <inertial>
-      <mass value="0.01"/>
-      <inertia ixx="0.0001" ixy="0" ixz="0" iyy="0.0001" iyz="0" izz="0.0001"/>
+      <mass value="0.01" />
+      <inertia ixx="0.0001" ixy="0" ixz="0" iyy="0.0001" iyz="0" izz="0.0001" />
     </inertial>
   </link>
   <joint name="right_track_visual_joint" type="fixed">
-    <parent link="base_link"/>
-    <child link="right_track_visual"/>
-    <origin xyz="0 ${-track_y_offset} ${track_z_offset}" rpy="0 0 0"/>
+    <parent link="base_link" />
+    <child link="right_track_visual" />
+    <origin xyz="0 ${-track_y_offset} ${track_z_offset}" rpy="0 0 0" />
   </joint>
   <!-- ==================== -->
@@ -145,27 +155,27 @@
   <!-- Left side wheels (3 wheels) -->
   <xacro:hidden_wheel name="left_front_wheel"
-                       x_pos="${wheel_front_x}"
-                       y_pos="${track_y_offset}"
-                       z_pos="${wheel_z}"/>
+    x_pos="${wheel_front_x}"
+    y_pos="${track_y_offset}"
+    z_pos="${wheel_z}" />
   <xacro:hidden_wheel name="left_mid_wheel"
-                       x_pos="${wheel_mid_x}"
-                       y_pos="${track_y_offset}"
-                       z_pos="${wheel_z}"/>
+    x_pos="${wheel_mid_x}"
+    y_pos="${track_y_offset}"
+    z_pos="${wheel_z}" />
   <xacro:hidden_wheel name="left_rear_wheel"
-                       x_pos="${wheel_rear_x}"
-                       y_pos="${track_y_offset}"
-                       z_pos="${wheel_z}"/>
+    x_pos="${wheel_rear_x}"
+    y_pos="${track_y_offset}"
+    z_pos="${wheel_z}" />
   <!-- Right side wheels (3 wheels) -->
   <xacro:hidden_wheel name="right_front_wheel"
-                       x_pos="${wheel_front_x}"
-                       y_pos="${-track_y_offset}"
-                       z_pos="${wheel_z}"/>
+    x_pos="${wheel_front_x}"
+    y_pos="${-track_y_offset}"
+    z_pos="${wheel_z}" />
   <xacro:hidden_wheel name="right_mid_wheel"
-                       x_pos="${wheel_mid_x}"
-                       y_pos="${-track_y_offset}"
-                       z_pos="${wheel_z}"/>
+    x_pos="${wheel_mid_x}"
+    y_pos="${-track_y_offset}"
+    z_pos="${wheel_z}" />
   <xacro:hidden_wheel name="right_rear_wheel"
-                       x_pos="${wheel_rear_x}"
-                       y_pos="${-track_y_offset}"
-                       z_pos="${wheel_z}"/>
+    x_pos="${wheel_rear_x}"
+    y_pos="${-track_y_offset}"
+    z_pos="${wheel_z}" />
 </robot>
