Commit message: URDF modifications, LiDAR modes, Docker setup

File: urdf/gazebo.xacro (robot description, xacro)
@@ -4,5 +4,4 @@
   <!-- GAZEBO FRICTION      -->
   <!-- ==================== -->
-  <!-- High friction for track wheels (critical for tracked robots) -->
   <xacro:macro name="wheel_friction" params="wheel_name">
     <gazebo reference="${wheel_name}">
@@ -34,9 +33,25 @@
     <material>Gazebo/Black</material>
   </gazebo>
+  <gazebo reference="gimbal_base_link">
+    <material>Gazebo/DarkGrey</material>
+  </gazebo>
+  <gazebo reference="gimbal_pan_link">
+    <material>Gazebo/DarkGrey</material>
+  </gazebo>
+  <gazebo reference="gimbal_tilt_link">
+    <material>Gazebo/DarkGrey</material>
+    <self_collide>false</self_collide>
+  </gazebo>
   <gazebo reference="gimbal_pan_link">
     <self_collide>false</self_collide>
   </gazebo>
-  <gazebo reference="gimbal_tilt_link">
-    <self_collide>false</self_collide>
+  <gazebo reference="camera_holder_link">
+    <material>Gazebo/DarkGrey</material>
+  </gazebo>
+  <gazebo reference="lidar_link">
+    <material>Gazebo/DarkGray</material>
+  </gazebo>
+  <gazebo reference="rifle_link">
+    <material>Gazebo/Black</material>
   </gazebo>
 </robot>

File: urdf/gazebo_control.xacro (robot description, xacro)
@@ -4,11 +4,7 @@
     <xacro:arg name="robot_ns" default="" />
     <xacro:property name="ns" value="$(arg robot_ns)" />
-    <!-- Topic prefix: /ns or empty for topics -->
     <xacro:property name="topic_prefix" value="${'/' + ns if ns != '' else ''}" />
-    <!-- Frame prefix: ns/ or empty for frame_ids (no leading slash) -->
     <xacro:property name="frame_prefix" value="${ns + '/' if ns != '' else ''}" />
-    <!-- ==================== -->
     <!-- DIFFERENTIAL DRIVE   -->
-    <!-- ==================== -->
     <gazebo>
         <plugin filename="gz-sim-diff-drive-system" name="gz::sim::systems::DiffDrive">
@@ -49,7 +45,5 @@
         </plugin>
     </gazebo>
-    <!-- ==================== -->
     <!-- GIMBAL CONTROLLERS   -->
-    <!-- ==================== -->
     <!-- Gimbal Pan Controller -->
     <gazebo>
@@ -58,7 +52,4 @@
             <joint_name>gimbal_pan_joint</joint_name>
             <topic>${topic_prefix}/gimbal/pan_cmd</topic>
-            <!-- <p_gain>10</p_gain>
-            <i_gain>0.1</i_gain>
-            <d_gain>0.5</d_gain> -->
             <p_gain>5</p_gain>
             <i_gain>0.0</i_gain>
@@ -72,7 +63,4 @@
             <joint_name>gimbal_tilt_joint</joint_name>
             <topic>${topic_prefix}/gimbal/tilt_cmd</topic>
-            <!-- <p_gain>10</p_gain>
-            <i_gain>0.1</i_gain>
-            <d_gain>0.5</d_gain> -->
             <p_gain>5</p_gain>
             <i_gain>0.0</i_gain>

File: urdf/gimbal.xacro (robot description, xacro)
@@ -1,12 +1,39 @@
 <?xml version="1.0"?>
 <robot xmlns:xacro="http://www.ros.org/wiki/xacro" name="gimbal">
-  <!-- Properties -->
-  <xacro:property name="pedestal_z" value="0.073" />
-  <xacro:property name="pan_z" value="0.194" />
-  <xacro:property name="tilt_z" value="0.211" />
-  <!-- ============ GIMBAL BASE (Pedestal) ============ -->
+  <!-- Gimbal Base dimensions(meters) -->
+  <xacro:property name="gimbal_base_x" value="0.155" />
+  <xacro:property name="gimbal_base_y" value="0.155" />
+  <xacro:property name="gimbal_base_z" value="0.073" />
+  <xacro:property name="gimbal_base_mass" value="0.5" />
+  <!-- Gimbal Pan dimensions(meters) -->
+  <xacro:property name="gimbal_pan_x" value="0.180" />
+  <xacro:property name="gimbal_pan_y" value="0.172" />
+  <xacro:property name="gimbal_pan_z" value="0.194" />
+  <xacro:property name="gimbal_pan_mass" value="0.8" />
+  <!-- Gimbal Tilt dimensions(meters) -->
+  <xacro:property name="gimbal_tilt_x" value="0.125" />
+  <xacro:property name="gimbal_tilt_y" value="0.256" />
+  <xacro:property name="gimbal_tilt_z" value="0.219" />
+  <xacro:property name="gimbal_tilt_mass" value="0.5" />
+  <!-- Joint offsets(meters) -->
+  <xacro:property name="pan_joint_z" value="0.133" />
+  <xacro:property name="tilt_joint_z" value="0.028" />
+  <!-- Gimbal Damping and Friction -->
+  <xacro:property name="gimbal_damping" value="5" />
+  <xacro:property name="gimbal_friction" value="0.1" />
+  <!-- Pan joint limits -->
+  <xacro:property name="pan_lower" value="${-pi}" />
+  <xacro:property name="pan_upper" value="${pi}" />
+  <xacro:property name="pan_effort" value="10" />
+  <xacro:property name="pan_velocity" value="1.0" />
+  <!-- Tilt joint limits -->
+  <xacro:property name="tilt_lower" value="${-pi/4}" />
+  <xacro:property name="tilt_upper" value="${pi/4}" />
+  <xacro:property name="tilt_effort" value="10" />
+  <xacro:property name="tilt_velocity" value="1.0" />
+  <!-- ============ BASE ============ -->
   <link name="gimbal_base_link">
     <visual>
-      <origin xyz="0 0 0" rpy="${pi} 0 0" />
+      <origin xyz="0 0 0" rpy="0 0 0" />
       <geometry>
         <mesh filename="package://tin3_bot/meshes/gimbal_base.dae" />
@@ -15,17 +42,17 @@
     <collision>
       <geometry>
-        <box size="0.155 0.155 0.073" />
+        <box size="${gimbal_base_x} ${gimbal_base_y} ${gimbal_base_z}" />
       </geometry>
     </collision>
     <inertial>
-      <mass value="0.5" />
-      <inertia ixx="0.001" ixy="0" ixz="0" iyy="0.001" iyz="0" izz="0.001" />
+      <mass value="${gimbal_base_mass}" />
+      <xacro:box_inertia m="${gimbal_base_mass}" x="${gimbal_base_x}" y="${gimbal_base_y}"
+        z="${gimbal_base_z}" />
     </inertial>
   </link>
-  <!-- ============ GIMBAL PAN (Big Box) ============ -->
+  <!-- ============ PAN ============ -->
   <link name="gimbal_pan_link">
     <visual>
-      <!-- <origin xyz="0 0 0" rpy="${pi} 0 0"/> -->
-      <origin xyz="0 0 0" rpy="${pi} 0 ${pi}" />
+      <origin xyz="0 0 0" rpy="0 0 0" />
       <geometry>
         <mesh filename="package://tin3_bot/meshes/gimbal_pan.dae" />
@@ -34,10 +61,11 @@
     <collision>
       <geometry>
-        <box size="0.15 0.15 0.15" />  <!-- Smaller -->
+        <box size="${gimbal_pan_x} ${gimbal_pan_y} ${gimbal_pan_z}" />
       </geometry>
     </collision>
     <inertial>
-      <mass value="0.8" />
-       <inertia ixx="0.003" ixy="0" ixz="0" iyy="0.003" iyz="0" izz="0.003" />
+      <mass value="${gimbal_pan_mass}" />
+      <xacro:box_inertia m="${gimbal_pan_mass}" x="${gimbal_pan_x}" y="${gimbal_pan_y}"
+        z="${gimbal_pan_z}" />
     </inertial>
   </link>
@@ -45,13 +73,13 @@
     <parent link="gimbal_base_link" />
     <child link="gimbal_pan_link" />
-    <origin xyz="0 0 ${pedestal_z/2 + pan_z/2}" rpy="0 0 0" />
+    <origin xyz="0 0 ${pan_joint_z}" rpy="0 0 0" />
     <axis xyz="0 0 1" />
-    <limit lower="${-pi}" upper="${pi}" effort="10" velocity="1.0" />
-    <dynamics damping="0.5" friction="0.1" />
+    <limit lower="${pan_lower}" upper="${pan_upper}" effort="${pan_effort}" velocity="${pan_velocity}" />
+    <dynamics damping="${gimbal_damping}" friction="${gimbal_friction}" />
   </joint>
-  <!-- ============ GIMBAL TILT (Head) ============ -->
+  <!-- ============ TILT ============ -->
   <link name="gimbal_tilt_link">
     <visual>
-      <origin xyz="0 0 0" rpy="${pi} 0 0" />
+      <origin xyz="0 0 0" rpy="0 0 0" />
       <geometry>
         <mesh filename="package://tin3_bot/meshes/gimbal_tilt.dae" />
@@ -60,10 +88,11 @@
     <collision>
       <geometry>
-        <box size="0.10 0.18 0.15" />
+        <box size="${gimbal_tilt_x} ${gimbal_tilt_y} ${gimbal_tilt_z}" />
       </geometry>
     </collision>
     <inertial>
-      <mass value="0.5" />
-      <inertia ixx="0.0023" ixy="0" ixz="0" iyy="0.0014" iyz="0" izz="0.0018" />
+      <mass value="${gimbal_tilt_mass}" />
+      <xacro:box_inertia m="${gimbal_tilt_mass}" x="${gimbal_tilt_x}" y="${gimbal_tilt_y}"
+        z="${gimbal_tilt_z}" />
     </inertial>
   </link>
@@ -71,81 +100,14 @@
     <parent link="gimbal_pan_link" />
     <child link="gimbal_tilt_link" />
-    <!-- <origin xyz="0 0 ${pan_z/2 + tilt_z/2}" rpy="0 0 0"/> -->
-    <!-- <origin xyz="0 0 ${pan_z/2}" rpy="0 0 0"/> -->
-    <origin xyz="0 0 0.01" rpy="0 0 0" />
+    <origin xyz="0 0 ${tilt_joint_z}" rpy="0 0 0" />
     <axis xyz="0 1 0" />
-    <limit lower="${-pi/4}" upper="${pi/4}" effort="10" velocity="1.0" />
-    <dynamics damping="0.5" friction="0.1" />
+    <limit lower="${tilt_lower}" upper="${tilt_upper}" effort="${tilt_effort}" velocity="${tilt_velocity}" />
+    <dynamics damping="${gimbal_damping}" friction="${gimbal_friction}" />
   </joint>
-  <!-- ============ RGB Camera Link ============ -->
-  <link name="gimbal_camera_link">
-    <visual>
-      <origin xyz="0 0 0" rpy="0 -1.5708 3.1416" />
-      <geometry>
-        <mesh filename="package://tin3_bot/meshes/camera.dae" />
-      </geometry>
-    </visual>
-    <!-- <collision>
-      <origin xyz="0 0 0" rpy="0 0 0" />
-      <geometry>
-        <mesh filename="package://tin3_bot/meshes/camera.dae" />
-      </geometry>
-    </collision> -->
-    <collision>
-      <origin xyz="0 0 0" rpy="0 0 0" />
-      <geometry>
-        <box size="0.055 0.064 0.123" />
-      </geometry>
-    </collision>
-    <inertial>
-      <origin xyz="0 0 0" rpy="0 0 0" />
-      <mass value="0.05" />
-      <inertia
-        ixx="1e-4" ixy="0.0" ixz="0.0"
-        iyy="1e-4" iyz="0.0"
-        izz="1e-4" />
-    </inertial>
-  </link>
-  <joint name="gimbal_camera_joint" type="fixed">
-    <parent link="gimbal_tilt_link" />
-    <child link="gimbal_camera_link" />
-    <origin xyz="0 -0.03 ${tilt_z/2+0.025}" rpy="0 0 0" />
-  </joint>
-  <!-- ============ IR Camera Link ============ -->
-  <link name="gimbal_ir_camera_link">
-    <visual>
-      <origin xyz="0 0 0" rpy="0 -1.5708 3.1416" />
-      <geometry>
-        <mesh filename="package://tin3_bot/meshes/camera.dae" />
-      </geometry>
-    </visual>
-    <collision>
-      <geometry>
-        <box size="0.055 0.064 0.123" />
-      </geometry>
-    </collision>
-    <inertial>
-      <mass value="0.05" />
-      <inertia ixx="0.0001" ixy="0" ixz="0" iyy="0.0001" iyz="0" izz="0.0001" />
-    </inertial>
-  </link>
-  <joint name="gimbal_ir_camera_joint" type="fixed">
-    <parent link="gimbal_tilt_link" />
-    <child link="gimbal_ir_camera_link" />
-    <origin xyz="0 0.03 ${tilt_z/2+0.025}" rpy="0 0 0" />
-  </joint>
-  <!-- RGB Camera Optical Frame -->
-  <link name="gimbal_camera_optical_frame" />
-  <joint name="gimbal_camera_optical_joint" type="fixed">
-    <parent link="gimbal_camera_link" />
-    <child link="gimbal_camera_optical_frame" />
-    <origin xyz="0 0 0" rpy="${-pi/2} 0 ${-pi/2}" />
-  </joint>
-  <!-- IR Camera Optical Frame -->
-  <link name="gimbal_ir_camera_optical_frame" />
-  <joint name="gimbal_ir_camera_optical_joint" type="fixed">
-    <parent link="gimbal_ir_camera_link" />
-    <child link="gimbal_ir_camera_optical_frame" />
-    <origin xyz="0 0 0" rpy="${-pi/2} 0 ${-pi/2}" />
+  <!-- ========== Gimbal Base to Baselink  ========== -->
+  <joint name="gimbal_base_joint" type="fixed">
+    <parent link="base_link" />
+    <child link="gimbal_base_link" />
+    <origin xyz="0.12  0  0.3395" rpy="0 0 0" />
   </joint>
 </robot>

File: urdf/robot.urdf.xacro (robot description, xacro)
@@ -1,195 +1,15 @@
 <?xml version="1.0"?>
 <robot xmlns:xacro="http://www.ros.org/wiki/xacro" name="tin3_bot">
+  <!-- Macros -->
+  <xacro:include filename="$(find tin3_bot)/urdf/macros.xacro" />
   <xacro:include filename="$(find tin3_bot)/urdf/materials.xacro" />
+  <!-- Robot body -->
+  <xacro:include filename="$(find tin3_bot)/urdf/chassis.xacro" />
+  <xacro:include filename="$(find tin3_bot)/urdf/gimbal.xacro" />
+  <xacro:include filename="$(find tin3_bot)/urdf/camera.xacro" />
+  <xacro:include filename="$(find tin3_bot)/urdf/rifle.xacro" />
+  <xacro:include filename="$(find tin3_bot)/urdf/sensors.xacro" />
+  <!-- Gazebo -->
   <xacro:include filename="$(find tin3_bot)/urdf/gazebo.xacro" />
   <xacro:include filename="$(find tin3_bot)/urdf/gazebo_control.xacro" />
-  <xacro:include filename="$(find tin3_bot)/urdf/gimbal.xacro" />
-  <xacro:include filename="$(find tin3_bot)/urdf/sensors.xacro" />
-  <!-- ==================== -->
-  <!-- PROPERTIES (meters)  -->
-  <!-- ==================== -->
-  <!-- Mesh scale: 0.001 to convert mm to meters -->
-  <xacro:property name="mesh_scale" value="1 1 1" />
-  <!-- Chassis dimensions (meters) -->
-  <xacro:property name="chassis_length" value="0.837" />
-  <xacro:property name="chassis_width" value="1.314" />
-  <xacro:property name="chassis_height" value="0.606" />
-  <xacro:property name="chassis_mass" value="20.0" />
-  <!-- Track offsets from base_link center (meters) -->
-  <xacro:property name="track_y_offset" value="0.35" />
-  <xacro:property name="track_z_offset" value="-0.22" />
-  <!-- Hidden wheel parameters -->
-  <xacro:property name="wheel_radius" value="0.12" />
-  <xacro:property name="wheel_width" value="0.10" />
-  <xacro:property name="wheel_mass" value="1.0" />
-  <!-- Wheel positions along track (X direction = front/back) -->
-  <xacro:property name="wheel_front_x" value="0.40" />
-  <xacro:property name="wheel_mid_x" value="0.0" />
-  <xacro:property name="wheel_rear_x" value="-0.40" />
-  <!-- Wheel Z position (below base_link origin) -->
-  <!-- <xacro:property name="wheel_z" value="-0.15"/> -->
-  <xacro:property name="wheel_z" value="-0.27" />
-  <!-- ==================== -->
-  <!-- MACROS               -->
-  <!-- ==================== -->
-  <!-- Macro for inertia of a box -->
-  <xacro:macro name="box_inertia" params="m x y z">
-    <inertia ixx="${m*(y*y+z*z)/12}" ixy="0" ixz="0"
-      iyy="${m*(x*x+z*z)/12}" iyz="0"
-      izz="${m*(x*x+y*y)/12}" />
-  </xacro:macro>
-  <!-- Macro for inertia of a cylinder -->
-  <xacro:macro name="cylinder_inertia" params="m r l">
-    <inertia ixx="${m*(3*r*r+l*l)/12}" ixy="0" ixz="0"
-      iyy="${m*(3*r*r+l*l)/12}" iyz="0"
-      izz="${m*r*r/2}" />
-  </xacro:macro>
-  <!-- Macro for hidden wheel -->
-  <xacro:macro name="hidden_wheel" params="name x_pos y_pos z_pos">
-    <link name="${name}">
-      <collision>
-        <origin xyz="0 0 0" rpy="${pi/2} 0 0" />
-        <geometry>
-          <cylinder radius="${wheel_radius}" length="${wheel_width}" />
-        </geometry>
-      </collision>
-      <inertial>
-        <origin xyz="0 0 0" rpy="0 0 0" />
-        <mass value="${wheel_mass}" />
-        <xacro:cylinder_inertia m="${wheel_mass}" r="${wheel_radius}" l="${wheel_width}" />
-      </inertial>
-    </link>
-    <joint name="${name}_joint" type="continuous">
-      <parent link="base_link" />
-      <child link="${name}" />
-      <origin xyz="${x_pos} ${y_pos} ${z_pos}" rpy="0 0 0" />
-      <axis xyz="0 1 0" />
-    </joint>
-  </xacro:macro>
-  <!-- ==================== -->
-  <!-- BASE FOOTPRINT       -->
-  <!-- ==================== -->
-  <link name="base_footprint" />
-  <joint name="base_footprint_joint" type="fixed">
-    <parent link="base_footprint" />
-    <child link="base_link" />
-    <!-- <origin xyz="0 0 0.27" rpy="0 0 0"/> -->
-    <origin xyz="0 0 0.387" rpy="0 0 0" />
-  </joint>
-  <!-- ==================== -->
-  <!-- BASE LINK (CHASSIS)  -->
-  <!-- ==================== -->
-  <link name="base_link">
-    <visual>
-      <origin xyz="0 0 0" rpy="0 0 ${pi/2}" />
-      <geometry>
-        <mesh filename="package://tin3_bot/meshes/chassis.dae" scale="${mesh_scale}" />
-      </geometry>
-      <material name="dark_gray" />
-    </visual>
-    <collision>
-      <origin xyz="0 0 0" rpy="0 0 0" />
-      <geometry>
-         <box size="1.32 0.55 0.49" />
-      </geometry>
-    </collision>
-    <inertial>
-      <origin xyz="0 0 0" rpy="0 0 0" />
-      <mass value="${chassis_mass}" />
-      <xacro:box_inertia m="${chassis_mass}" x="${chassis_length}" y="${chassis_width}"
-        z="${chassis_height}" />
-    </inertial>
-  </link>
-  <!-- ==================== -->
-  <!-- Gimbal Joint        -->
-  <!-- ==================== -->
-  <joint name="gimbal_base_joint" type="fixed">
-    <parent link="base_link" />
-    <child link="gimbal_base_link" />
-    <origin xyz="0.1  0  0.303" rpy="0 0 0" />
-  </joint>
-  <!-- ==================== -->
-  <!-- TRACK VISUALS        -->
-  <!-- ==================== -->
-  <!-- Left Track Visual -->
-  <link name="left_track_visual">
-    <visual>
-      <origin xyz="0 0 0" rpy="0 0 ${-pi/2}" />
-      <geometry>
-        <mesh filename="package://tin3_bot/meshes/left_track.dae" scale="${mesh_scale}" />
-      </geometry>
-      <material name="dark_gray" />
-    </visual>
-    <collision>
-      <origin xyz="0 0 0" rpy="0 0 0" />
-      <geometry>
-        <!-- <box size="0.8 0.15 0.24" /> -->
-          <box size="1.22 0.154 0.33" />
-      </geometry>
-    </collision>
-    <inertial>
-      <mass value="0.01" />
-      <inertia ixx="0.0001" ixy="0" ixz="0" iyy="0.0001" iyz="0" izz="0.0001" />
-    </inertial>
-  </link>
-  <joint name="left_track_visual_joint" type="fixed">
-    <parent link="base_link" />
-    <child link="left_track_visual" />
-    <origin xyz="0 ${track_y_offset} ${track_z_offset}" rpy="0 0 0" />
-  </joint>
-  <!-- Right Track Visual -->
-  <link name="right_track_visual">
-    <visual>
-      <origin xyz="0 0 0" rpy="0 0 ${-pi/2}" />
-      <geometry>
-        <mesh filename="package://tin3_bot/meshes/right_track.dae" scale="${mesh_scale}" />
-      </geometry>
-      <material name="dark_gray" />
-    </visual>
-    <collision>
-      <origin xyz="0 0 0" rpy="0 0 0" />
-      <geometry>
-        <!-- <box size="0.8 0.15 0.24" /> -->
-        <box size="1.22 0.154 0.33" />
-      </geometry>
-    </collision>
-    <inertial>
-      <mass value="0.01" />
-      <inertia ixx="0.0001" ixy="0" ixz="0" iyy="0.0001" iyz="0" izz="0.0001" />
-    </inertial>
-  </link>
-  <joint name="right_track_visual_joint" type="fixed">
-    <parent link="base_link" />
-    <child link="right_track_visual" />
-    <origin xyz="0 ${-track_y_offset} ${track_z_offset}" rpy="0 0 0" />
-  </joint>
-  <!-- ==================== -->
-  <!-- HIDDEN WHEELS        -->
-  <!-- ==================== -->
-  <!-- Left side wheels (3 wheels) -->
-  <xacro:hidden_wheel name="left_front_wheel"
-    x_pos="${wheel_front_x}"
-    y_pos="${track_y_offset}"
-    z_pos="${wheel_z}" />
-  <xacro:hidden_wheel name="left_mid_wheel"
-    x_pos="${wheel_mid_x}"
-    y_pos="${track_y_offset}"
-    z_pos="${wheel_z}" />
-  <xacro:hidden_wheel name="left_rear_wheel"
-    x_pos="${wheel_rear_x}"
-    y_pos="${track_y_offset}"
-    z_pos="${wheel_z}" />
-  <!-- Right side wheels (3 wheels) -->
-  <xacro:hidden_wheel name="right_front_wheel"
-    x_pos="${wheel_front_x}"
-    y_pos="${-track_y_offset}"
-    z_pos="${wheel_z}" />
-  <xacro:hidden_wheel name="right_mid_wheel"
-    x_pos="${wheel_mid_x}"
-    y_pos="${-track_y_offset}"
-    z_pos="${wheel_z}" />
-  <xacro:hidden_wheel name="right_rear_wheel"
-    x_pos="${wheel_rear_x}"
-    y_pos="${-track_y_offset}"
-    z_pos="${wheel_z}" />
 </robot>
