Commit message: URDF modifications, LiDAR modes, Docker setup

File: urdf/sensors.xacro (robot description, xacro)
@@ -1,5 +1,5 @@
 <?xml version="1.0"?>
 <robot xmlns:xacro="http://www.ros.org/wiki/xacro" name="tin3_bot">
-    <!-- Add namespace properties at top of sensors.xacro -->
+    <!-- Namespace configuration for multi-robot support -->
     <xacro:arg name="robot_ns" default="" />
     <xacro:property name="ns" value="$(arg robot_ns)" />
@@ -7,8 +7,42 @@
     <xacro:property name="frame_prefix" value="${ns + '/' if ns != '' else ''}" />
     <!-- ==================== -->
-    <!-- GPS SENSOR           -->
+    <!-- LiDAR Configuration  -->
     <!-- ==================== -->
-    <xacro:property name="gps_xyz" value="-0.4 0 0.35" />
-    <xacro:property name="gps_rpy" value="0 0 0" />
+    <!-- Mode: full (single robot), half (2-4 robots), low (8+ robots) -->
+    <xacro:arg name="lidar_mode" default="full" />
+    <xacro:property name="lidar_mode" value="$(arg lidar_mode)" />
+    <!-- Full resolution (27,648 points/scan) -->
+    <xacro:property name="lidar_h_samples_full" value="192" />
+    <xacro:property name="lidar_v_samples_full" value="144" />
+    <xacro:property name="lidar_update_rate_full" value="10" />
+    <!-- Half resolution (6,912 points/scan) -->
+    <xacro:property name="lidar_h_samples_half" value="96" />
+    <xacro:property name="lidar_v_samples_half" value="72" />
+    <xacro:property name="lidar_update_rate_half" value="10" />
+    <!-- Low resolution (1,728 points/scan) -->
+    <xacro:property name="lidar_h_samples_low" value="48" />
+    <xacro:property name="lidar_v_samples_low" value="36" />
+    <xacro:property name="lidar_update_rate_low" value="5" />
+    <!-- Select based on mode -->
+    <xacro:if value="${lidar_mode == 'full'}">
+        <xacro:property name="lidar_h_samples" value="${lidar_h_samples_full}" />
+        <xacro:property name="lidar_v_samples" value="${lidar_v_samples_full}" />
+        <xacro:property name="lidar_update_rate" value="${lidar_update_rate_full}" />
+    </xacro:if>
+    <xacro:if value="${lidar_mode == 'half'}">
+        <xacro:property name="lidar_h_samples" value="${lidar_h_samples_half}" />
+        <xacro:property name="lidar_v_samples" value="${lidar_v_samples_half}" />
+        <xacro:property name="lidar_update_rate" value="${lidar_update_rate_half}" />
+    </xacro:if>
+    <xacro:if value="${lidar_mode == 'low'}">
+        <xacro:property name="lidar_h_samples" value="${lidar_h_samples_low}" />
+        <xacro:property name="lidar_v_samples" value="${lidar_v_samples_low}" />
+        <xacro:property name="lidar_update_rate" value="${lidar_update_rate_low}" />
+    </xacro:if>
+    <!-- LiDAR dimensions (for reference) -->
+    <xacro:property name="lidar_x" value="0.063" />
+    <xacro:property name="lidar_y" value="0.175" />
+    <xacro:property name="lidar_z" value="0.118" />
+    <!-- GPS LINK -->
     <link name="gps_link">
         <inertial>
@@ -21,36 +55,7 @@
         <parent link="base_link" />
         <child link="gps_link" />
-        <origin xyz="${gps_xyz}" rpy="${gps_rpy}" />
+        <origin xyz="-0.4 0 0.35" rpy="0 0 0" />
     </joint>
-    <gazebo reference="gps_link">
-        <sensor name="gps_sensor" type="navsat">
-            <always_on>true</always_on>
-            <update_rate>5</update_rate>
-            <!-- <topic>/gps/fix</topic> -->
-            <!-- <gz_frame_id>gps_link</gz_frame_id> -->
-            <topic>${topic_prefix}/gps/fix</topic>
-            <gz_frame_id>${frame_prefix}gps_link</gz_frame_id>
-            <navsat>
-                <position_sensing>
-                    <horizontal>
-                        <noise type="gaussian">
-                            <mean>0.0</mean>
-                            <stddev>0.00001</stddev> <!-- ~1 meter in degrees -->
-                        </noise>
-                    </horizontal>
-                    <vertical>
-                        <noise type="gaussian">
-                            <mean>0.0</mean>
-                            <stddev>2.0</stddev> <!-- 2m altitude - this is OK -->
-                        </noise>
-                    </vertical>
-                </position_sensing>
-            </navsat>
-        </sensor>
-    </gazebo>
-    <!-- ==================== -->
-    <!-- IMU SENSOR           -->
-    <!-- ==================== -->
-    <xacro:property name="imu_xyz" value="0 0 0.05" />
+    <!-- IMU LINK -->
     <link name="imu_link">
         <inertial>
@@ -62,80 +67,18 @@
         <parent link="base_link" />
         <child link="imu_link" />
-        <origin xyz="${imu_xyz}" rpy="0 0 0" />
+        <origin xyz="0 0 0.05" rpy="0 0 0" />
     </joint>
-    <!-- IMU Gazebo Plugin (Harmonic) -->
-    <gazebo reference="imu_link">
-        <sensor name="imu_sensor" type="imu">
-            <always_on>true</always_on>
-            <update_rate>100</update_rate>
-            <!-- <topic>/imu/data</topic> -->
-            <!-- <gz_frame_id>imu_link</gz_frame_id> -->
-            <topic>${topic_prefix}/imu/data</topic>
-            <gz_frame_id>${frame_prefix}imu_link</gz_frame_id>
-            <imu>
-                <angular_velocity>
-                    <x>
-                        <noise type="gaussian">
-                            <mean>0.0</mean>
-                            <stddev>0.0002</stddev>
-                        </noise>
-                    </x>
-                    <y>
-                        <noise type="gaussian">
-                            <mean>0.0</mean>
-                            <stddev>0.0002</stddev>
-                        </noise>
-                    </y>
-                    <z>
-                        <noise type="gaussian">
-                            <mean>0.0</mean>
-                            <stddev>0.0002</stddev>
-                        </noise>
-                    </z>
-                </angular_velocity>
-                <linear_acceleration>
-                    <x>
-                        <noise type="gaussian">
-                            <mean>0.0</mean>
-                            <stddev>0.017</stddev>
-                        </noise>
-                    </x>
-                    <y>
-                        <noise type="gaussian">
-                            <mean>0.0</mean>
-                            <stddev>0.017</stddev>
-                        </noise>
-                    </y>
-                    <z>
-                        <noise type="gaussian">
-                            <mean>0.0</mean>
-                            <stddev>0.017</stddev>
-                        </noise>
-                    </z>
-                </linear_acceleration>
-            </imu>
-        </sensor>
-    </gazebo>
-    <!-- ==================== -->
-    <!-- LiDAR SENSOR           -->
-    <!-- ==================== -->
-    <xacro:property name="lidar_xyz" value="0.626 -0.01 -0.06" />
-    <xacro:property name="mesh_scale" value="1 1 1" />
+    <!-- LiDAR LINK -->
     <link name="lidar_link">
         <visual>
-            <origin xyz="0 0 0" rpy="${pi/2} 0 ${-pi/2}" />
+            <origin xyz="0 0 0" rpy="0 0 0" />
             <geometry>
-                <mesh filename="package://tin3_bot/meshes/lidar.dae" scale="${mesh_scale}" />
+                <mesh filename="package://tin3_bot/meshes/lidar.dae" scale="1 1 1" />
             </geometry>
             <material name="dark_gray" />
         </visual>
-        <collision>
-            <geometry>
-                <cylinder radius="0.045" length="0.03" />
-            </geometry>
-        </collision>
         <inertial>
             <mass value="0.5" />
-            <inertia ixx="0.001" ixy="0" ixz="0" iyy="0.001" iyz="0" izz="0.001" />
+            <inertia ixx="0.0001" ixy="0" ixz="0" iyy="0.0001" iyz="0" izz="0.0001" />
         </inertial>
     </link>
@@ -143,10 +86,36 @@
         <parent link="base_link" />
         <child link="lidar_link" />
-        <origin xyz="${lidar_xyz}" rpy="0 0 0" />
+        <origin xyz="0.626 -0.01 -0.06" rpy="0 0 0" />
     </joint>
+    <!-- GPS SENSOR -->
+    <gazebo reference="gps_link">
+        <sensor name="gps_sensor" type="navsat">
+            <always_on>true</always_on>
+            <update_rate>5</update_rate>
+            <topic>${topic_prefix}/gps/fix</topic>
+            <gz_frame_id>${frame_prefix}gps_link</gz_frame_id>
+            <navsat>
+                <position_sensing>
+                    <horizontal>
+                        <noise type="gaussian">
+                            <mean>0.0</mean>
+                            <stddev>0.00001</stddev> <!-- ~1 meter in degrees -->
+                        </noise>
+                    </horizontal>
+                    <vertical>
+                        <noise type="gaussian">
+                            <mean>0.0</mean>
+                            <stddev>2.0</stddev> <!-- 2m altitude - this is OK -->
+                        </noise>
+                    </vertical>
+                </position_sensing>
+            </navsat>
+        </sensor>
+    </gazebo>
+    <!-- LiDAR SENSOR -->
     <gazebo reference="lidar_link">
         <sensor name="lidar_sensor" type="gpu_lidar">
             <always_on>true</always_on>
-            <update_rate>10</update_rate>
+            <update_rate>${lidar_update_rate}</update_rate>
             <topic>${topic_prefix}/scan</topic>
             <gz_frame_id>${frame_prefix}lidar_link</gz_frame_id>
@@ -154,6 +123,5 @@
                 <scan>
                     <horizontal>
-                        <!-- FOV: 120° / 0.625° = 192 samples -->
-                        <samples>192</samples>
+                        <samples>${lidar_h_samples}</samples>
                         <resolution>1</resolution>
                         <min_angle>-1.0472</min_angle>  <!-- -60° -->
@@ -161,6 +129,5 @@
                     </horizontal>
                     <vertical>
-                        <!-- FOV: 90° with 144 lines (per spec) -->
-                        <samples>144</samples>
+                        <samples>${lidar_v_samples}</samples>
                         <resolution>1</resolution>
                         <min_angle>-0.7854</min_angle>  <!-- -45° -->
@@ -170,5 +137,5 @@
                 <range>
                     <min>0.1</min>
-                    <max>30.0</max>      <!-- 30m @ 10% reflectivity -->
+                    <max>30.0</max>
                     <resolution>0.01</resolution>
                 </range>
@@ -182,57 +149,53 @@
         </sensor>
     </gazebo>
-    <!-- ==================== -->
-    <!-- RGB CAMERA SENSOR    -->
-    <!-- ==================== -->
-    <gazebo reference="gimbal_camera_link">
-        <sensor name="rgb_camera" type="camera">
+    <!-- IMU SENSOR -->
+    <gazebo reference="imu_link">
+        <sensor name="imu_sensor" type="imu">
             <always_on>true</always_on>
-            <update_rate>30</update_rate>
-            <!-- <topic>/camera/image_raw</topic> -->
-            <!-- <gz_frame_id>gimbal_camera_link</gz_frame_id> -->
-            <topic>${topic_prefix}/camera/image_raw</topic>
-            <gz_frame_id>${frame_prefix}gimbal_camera_link</gz_frame_id>
-            <camera>
-                <horizontal_fov>1.047</horizontal_fov>
-                <image>
-                    <width>640</width>
-                    <height>480</height>
-                    <format>R8G8B8</format>
-                </image>
-                <clip>
-                    <near>0.1</near>
-                    <far>100</far>
-                </clip>
-                <noise>
-                    <type>gaussian</type>
-                    <mean>0.0</mean>
-                    <stddev>0.007</stddev>
-                </noise>
-            </camera>
-        </sensor>
-    </gazebo>
-    <!-- ==================== -->
-    <!-- IR CAMERA SENSOR     -->
-    <!-- ==================== -->
-    <gazebo reference="gimbal_ir_camera_link">
-        <sensor name="ir_camera" type="camera">
-            <always_on>true</always_on>
-            <update_rate>30</update_rate>
-            <!-- <topic>/ir/image_raw</topic> -->
-            <!-- <gz_frame_id>gimbal_ir_camera_link</gz_frame_id> -->
-            <topic>${topic_prefix}/ir/image_raw</topic>
-            <gz_frame_id>${frame_prefix}gimbal_ir_camera_link</gz_frame_id>
-            <camera>
-                <horizontal_fov>1.047</horizontal_fov>
-                <image>
-                    <width>640</width>
-                    <height>480</height>
-                    <format>L8</format>
-                </image>
-                <clip>
-                    <near>0.1</near>
-                    <far>100</far>
-                </clip>
-            </camera>
+            <update_rate>100</update_rate>
+            <topic>${topic_prefix}/imu/data</topic>
+            <gz_frame_id>${frame_prefix}imu_link</gz_frame_id>
+            <imu>
+                <angular_velocity>
+                    <x>
+                        <noise type="gaussian">
+                            <mean>0.0</mean>
+                            <stddev>0.0002</stddev>
+                        </noise>
+                    </x>
+                    <y>
+                        <noise type="gaussian">
+                            <mean>0.0</mean>
+                            <stddev>0.0002</stddev>
+                        </noise>
+                    </y>
+                    <z>
+                        <noise type="gaussian">
+                            <mean>0.0</mean>
+                            <stddev>0.0002</stddev>
+                        </noise>
+                    </z>
+                </angular_velocity>
+                <linear_acceleration>
+                    <x>
+                        <noise type="gaussian">
+                            <mean>0.0</mean>
+                            <stddev>0.017</stddev>
+                        </noise>
+                    </x>
+                    <y>
+                        <noise type="gaussian">
+                            <mean>0.0</mean>
+                            <stddev>0.017</stddev>
+                        </noise>
+                    </y>
+                    <z>
+                        <noise type="gaussian">
+                            <mean>0.0</mean>
+                            <stddev>0.017</stddev>
+                        </noise>
+                    </z>
+                </linear_acceleration>
+            </imu>
         </sensor>
     </gazebo>
