Commit message: verify(RP+LS): robot model, physics, all sensors verified (17/46 tasks)

File: tin3_description/urdf/camera.xacro (robot description, xacro)
@@ -81,5 +81,5 @@
             <always_on>true</always_on>
             <update_rate>30</update_rate>
-            <topic>${topic_prefix}/camera/image_raw</topic>
+            <topic>${topic_prefix}/rgb_camera/image_raw</topic>
             <gz_frame_id>${frame_prefix}rgb_camera_link</gz_frame_id>
             <camera>
@@ -107,5 +107,5 @@
             <always_on>true</always_on>
             <update_rate>30</update_rate>
-            <topic>${topic_prefix}/ir/image_raw</topic>
+            <topic>${topic_prefix}/ir_camera/image_raw</topic>
             <gz_frame_id>${frame_prefix}ir_camera_link</gz_frame_id>
             <camera>

File: tin3_description/urdf/chassis.xacro (robot description, xacro)
@@ -12,4 +12,7 @@
   <xacro:property name="track_height" value="0.334" />
   <xacro:property name="track_mass" value="0.01" />
+  <!-- Track collision (upper portion only - clears hidden wheels) -->
+  <xacro:property name="track_collision_height" value="0.297" />
+  <xacro:property name="track_collision_z_offset" value="0.019" />
   <!-- Track offsets from base_link center (meters) -->
   <xacro:property name="track_y_offset" value="0.35" />
@@ -71,9 +74,10 @@
       <material name="dark_gray" />
     </visual>
-    <!-- <collision>
+    <collision>
+      <origin xyz="0 0 ${track_collision_z_offset}" rpy="0 0 0" />
       <geometry>
-        <box size="${track_length} ${track_width} ${track_height}" />
+        <box size="${track_length} ${track_width} ${track_collision_height}" />
       </geometry>
-    </collision> -->
+    </collision>
     <inertial>
       <mass value="${track_mass}" />
@@ -96,9 +100,10 @@
       <material name="dark_gray" />
     </visual>
-    <!-- <collision>
+    <collision>
+      <origin xyz="0 0 ${track_collision_z_offset}" rpy="0 0 0" />
       <geometry>
-        <box size="${track_length} ${track_width} ${track_height}" />
+        <box size="${track_length} ${track_width} ${track_collision_height}" />
       </geometry>
-    </collision> -->
+    </collision>
     <inertial>
       <mass value="${track_mass}" />

File: tin3_description/urdf/gazebo_control.xacro (robot description, xacro)
@@ -25,4 +25,6 @@
             <min_linear_acceleration>-2.5</min_linear_acceleration>
             <min_angular_acceleration>-3</min_angular_acceleration>
+            <max_velocity>1.94</max_velocity>
+            <min_velocity>-1.94</min_velocity>
             <!-- Topics with namespace -->
             <topic>${topic_prefix}/cmd_vel</topic>

File: tin3_description/urdf/sensors.xacro (robot description, xacro)
@@ -44,4 +44,8 @@
     <xacro:property name="lidar_y" value="0.175" />
     <xacro:property name="lidar_z" value="0.118" />
+    <!-- LiDAR mount height above base_link (spec: 0.50m above ground) -->
+    <xacro:property name="lidar_z_offset" value="0.113" />
+    <!-- LiDAR tilt to meet 0.25m ground scan requirement -->
+    <xacro:property name="lidar_pitch" value="-0.272" />  <!-- -15.6° forward tilt in radians -->
     <!-- GPS LINK -->
     <link name="gps_link">
@@ -87,5 +91,6 @@
             <parent link="base_link" />
             <child link="lidar_link" />
-            <origin xyz="0.626 -0.01 -0.06" rpy="0 0 0" />
+            <!-- <origin xyz="0.626 -0.01 -0.06" rpy="0 0 0" /> before -->
+            <origin xyz="0.626 -0.01 ${lidar_z_offset}" rpy="0 ${lidar_pitch} 0" />
         </joint>
     </xacro:if>
